File: board/chrimbus2023.kicad_pcb (KiCad board)
At the start: 2 copper layers, 69.5 x 94 mm, 0 parts

Commit message: almost done
Parts:
- added C1: 1uF, Capacitor_SMD:C_0402_1005Metric, F.Cu at (79.5, 142.3)
- added C10: 1uF, Capacitor_SMD:C_0402_1005Metric, F.Cu at (82.2, 114.2)
- added C11: 1uF, Capacitor_SMD:C_0402_1005Metric, F.Cu at (73.0, 119.1)
- added C12: 1uF, Capacitor_SMD:C_0402_1005Metric, F.Cu at (82.3, 111.6)
- added C2: 1uF, Capacitor_SMD:C_0402_1005Metric, F.Cu at (77.7, 140.0)
- added C3: 1uF, Capacitor_SMD:C_0402_1005Metric, F.Cu at (79.9, 138.0)
- added C4: 1uF, Capacitor_SMD:C_0402_1005Metric, F.Cu at (69.3, 138.6)
- added C5: 1uF, Capacitor_SMD:C_0402_1005Metric, F.Cu at (78.8, 126.1)
- added C6: 1uF, Capacitor_SMD:C_0402_1005Metric, F.Cu at (79.7, 131.3)
- added C7: 1uF, Capacitor_SMD:C_0402_1005Metric, F.Cu at (68.4, 132.9)
- added C8: 0.1uF, Capacitor_SMD:C_0402_1005Metric, F.Cu at (79.3, 129.7)
- added C9: 0.1uF, Capacitor_SMD:C_0402_1005Metric, F.Cu at (76.6, 137.1)
- added G***: LOGO, silk:art, F.Cu at (98.0, 111.5)
- added G1: SJK_2NXX, Oscillator:Oscillator_SMD_ECS_2520MV-xxx-xx-4Pin_2.5x2.0mm, F.Cu at (68.1, 136.2)
- added J1: USB_A, toolbox-connector:usb-PCB, F.Cu at (74.5, 158.3)
- added R1: 10K, Resistor_SMD:R_0402_1005Metric, F.Cu at (79.3, 127.7)
- added R2: 12K, Resistor_SMD:R_0402_1005Metric, F.Cu at (69.7, 132.9)
- added R3: 10K, Resistor_SMD:R_0402_1005Metric, F.Cu at (69.0, 129.5)
- added R4: 10K, Resistor_SMD:R_0402_1005Metric, F.Cu at (72.0, 135.2)
- added R5: 10K, Resistor_SMD:R_0402_1005Metric, F.Cu at (69.9, 127.3)
- added U1: TLV7111833DDSER, Package_SON:WSON-6_1.5x1.5mm_P0.5mm, F.Cu at (79.5, 140.0)
- added U2: USBLC6-2P6, Package_TO_SOT_SMD:SOT-666, F.Cu at (73.8, 141.0)
- added U3: USB2240, Package_DFN_QFN:QFN-36-1EP_6x6mm_P0.5mm_EP4.1x4.1mm_ThermalVias, F.Cu at (74.7, 130.4)
- added U4: eMMC, toolbox-memory:BGA153C50P14X14_1100X1000X80, F.Cu at (74.7, 111.3)
Routing:
- net +3.3V: track 0.00 -> 81.5 mm, vias 0 -> 11
- net GND: track 0.00 -> 65.4 mm, vias 0 -> 19
- net +1V8: track 0.00 -> 58.7 mm, vias 0 -> 5
- net Net-(U3-SD_D7): track 0.00 -> 46.3 mm, vias 0 -> 3
- net Net-(U3-SD_D1): track 0.00 -> 44.8 mm, vias 0 -> 4
- net Net-(U3-SD_D0): track 0.00 -> 38.5 mm, vias 0 -> 2
- net Net-(U3-SD_D6): track 0.00 -> 36.0 mm, vias 0 -> 6
- net Net-(U3-SD_CLK): track 0.00 -> 33.3 mm, vias 0 -> 4
- net Net-(U3-SD_D5): track 0.00 -> 30.4 mm, vias 0 -> 2
- net Net-(U3-SD_CMD): track 0.00 -> 24.5 mm, vias 0 -> 2
- net VBUS: track 0.00 -> 20.8 mm
- net Net-(U3-SD_D2): track 0.00 -> 18.9 mm
- net Net-(U3-CRD_PWR): track 0.00 -> 17.5 mm, vias 0 -> 2
- net Net-(U3-SD_D4): track 0.00 -> 17.1 mm, vias 0 -> 2
- net Net-(U3-SD_D3): track 0.00 -> 15.0 mm
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- added copper zone on B.Cu, net GND
- added copper zone on F.Cu, net GND

Commit message: final
Parts:
- added D1: LED, LED_SMD:LED_1206_3216Metric_Pad1.42x1.75mm_HandSolder, F.Cu at (74.6, 102.1)
- added H1: MountingHole, MountingHole:MountingHole_3.2mm_M3, F.Cu at (90.4, 68.3)
- moved G*** 0.18 mm to (98.1, 111.3)
Routing:
- net Net-(D1-A): track 0.00 -> 53.0 mm
- net /D-: track 14.8 -> 12.0 mm
- net GND: track 65.4 -> 67.3 mm, vias 19 -> 22
- net +3.3V: track 81.5 -> 80.7 mm
- net +1V8: track 58.7 -> 58.6 mm, vias 5 -> 4
- net Net-(U3-SD_D7): vias 3 -> 2

Commit message: 2024
Parts:
- G***: footprint silk:art -> silk:art_2024
